File: Estacion/Estacion.kicad_pcb (KiCad board)
At the start: 2 copper layers, 120 x 62.2 mm, 12 parts, among them SW1 SW_Push, U4 WeMos_S2_mini, U5 DHT22, U6 FN-M16P

Commit message: Emily me pega
Parts:
- D3, D4, D5: footprint LED_THT:LED_D5.0mm-4_RGB -> LED_THT:LED_D5.0mm-4_RGB_Wide_Pins
- moved U6 96.8 mm to (76.0, 102.0), turned to 180 degrees
- moved D5 51.9 mm to (135.0, 105.3)
- moved D4 38.0 mm to (135.1, 96.4)
- moved R2 34.0 mm to (113.3, 56.5)
- moved R3 34.0 mm to (115.3, 60.8)
- moved D3 28.1 mm to (135.2, 87.8)
- moved U4 22.0 mm to (94.1, 86.6)
- moved BMP280 21.5 mm to (178.2, 102.6)
- moved U5 19.8 mm to (150.0, 99.7)
- moved R1 19.6 mm to (152.6, 81.4)
- moved D1 6.01 mm to (136.0, 68.0)
Routing:
- net Net-(U4-GPIO5): track 181.5 -> 81.1 mm
- net Net-(U4-GPIO11): track 105.8 -> 15.7 mm, vias 1 -> 0
- net Net-(U4-GPIO12): track 107.9 -> 19.3 mm
- net Net-(U4-GPIO14): track 130.4 -> 67.3 mm
- net Net-(U4-GPIO3): track 105.1 -> 51.4 mm
- net Net-(D5-BK): track 93.5 -> 49.5 mm, vias 0 -> 1
- net /SCL: track 195.6 -> 156.9 mm, vias 0 -> 1
- net /SDA: track 128.6 -> 159.0 mm
- net +5V: track 71.5 -> 43.7 mm, vias 0 -> 1
- net Net-(D4-GK): track 71.3 -> 45.4 mm
- net Net-(D5-RK): track 82.2 -> 56.5 mm
- net +3V3: track 204.1 -> 188.6 mm
- net Net-(D3-BK): track 61.5 -> 46.4 mm, vias 0 -> 1
- net Net-(D4-BK): track 30.1 -> 17.3 mm
- net Net-(D5-GK): track 31.9 -> 25.2 mm
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Other:
- board size 120 x 62.2 mm -> 120 x 64.1 mm

Commit message: Hola pipol de youtube
Changed lines of the file:
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@@
 		(capping no)
 		(filling no)
-		(zone_defaults)
 		(pcbplotparams
 			(layerselection 0x00000000_00000000_55555555_5755f5ff)
@@
 	(gr_rect
 		(start 64.897 52.07)
-		(end 184.912 116.12)
+		(end 184.88 116.12)
 		(stroke
 			(width 0.2)
