File: Estacion/Estacion.kicad_pcb (KiCad board)
At the start: 2 copper layers, 120 x 64.1 mm, 12 parts, among them SW1 SW_Push, U4 WeMos_S2_mini, U5 DHT22, U6 FN-M16P

Commit message: Arreglar error por culpa del tru hole malo ese de yahiko
Parts:
- R1: moved to B.Cu
- turned R1 to 0 degrees
Routing:
- net GND: track 253.9 -> 14.5 mm, vias 1 -> 3
- net Net-(D3-BK): track 46.4 -> 169.4 mm, vias 1 -> 5
- net Net-(D5-BK): track 49.5 -> 63.5 mm
- net +3V3: track 188.6 -> 200.8 mm, vias 0 -> 4
- net Net-(U4-GPIO5): track 81.1 -> 92.8 mm, vias 0 -> 2
- net /SCL: track 156.9 -> 163.9 mm, vias 1 -> 2
- net +5V: track 43.7 -> 49.9 mm, vias 1 -> 2
- net Net-(D3-RK): track 50.0 -> 54.5 mm, vias 0 -> 3
- net Net-(U4-GPIO14): track 67.3 -> 71.6 mm, vias 1 -> 2
- net /SDA: track 159.0 -> 155.5 mm, vias 0 -> 1
- net Net-(D5-RK): track 56.5 -> 53.6 mm, vias 0 -> 1
- net Net-(D3-GK): track 17.2 -> 15.1 mm
- net Net-(D4-RK): track 23.7 -> 22.1 mm, vias 0 -> 1
- net Net-(D4-GK): track 45.4 -> 46.8 mm
- net Net-(D4-BK): track 17.3 -> 18.6 mm, vias 0 -> 1
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- added copper zone on F.Cu, net GND

Commit message: ?
Parts:
- added J1: Conn_01x02_Pin, Connector_PinHeader_2.54mm:PinHeader_1x02_P2.54mm_Vertical, F.Cu at (181.0, 70.2)
- added R10: 220, Resistor_SMD:R_0805_2012Metric_Pad1.20x1.40mm_HandSolder, F.Cu at (141.0, 97.8)
- added R11: 150, Resistor_SMD:R_0805_2012Metric_Pad1.20x1.40mm_HandSolder, B.Cu at (119.8, 89.0)
- added R12: 150, Resistor_SMD:R_0805_2012Metric_Pad1.20x1.40mm_HandSolder, B.Cu at (118.2, 109.8)
- added R4: 220, Resistor_SMD:R_0805_2012Metric_Pad1.20x1.40mm_HandSolder, F.Cu at (127.7, 112.1)
- added R5: 150, Resistor_SMD:R_0805_2012Metric_Pad1.20x1.40mm_HandSolder, F.Cu at (124.2, 98.0)
- added R6: 150, Resistor_SMD:R_0805_2012Metric_Pad1.20x1.40mm_HandSolder, B.Cu at (107.0, 103.2)
- added R7: 150, Resistor_SMD:R_0805_2012Metric_Pad1.20x1.40mm_HandSolder, F.Cu at (140.0, 91.8)
- added R8: 150, Resistor_SMD:R_0805_2012Metric_Pad1.20x1.40mm_HandSolder, F.Cu at (121.8, 89.5)
- added R9: 220, Resistor_SMD:R_0805_2012Metric_Pad1.20x1.40mm_HandSolder, F.Cu at (126.8, 92.8)
Connections:
- U4 pad 13: Net-(D3-GK) -> Net-(U4-GPIO33)
- U4 pad 14: Net-(D4-RK) -> Net-(U4-GPIO35)
- U4 pad 15: Net-(D4-BK) -> Net-(U4-GPIO37)
- U4 pad 16: Net-(D5-GK) -> Net-(U4-GPIO39)
- U4 pad 28: Net-(D3-RK) -> Net-(U4-GPIO21)
- U4 pad 29: Net-(D3-BK) -> Net-(U4-GPIO34)
- U4 pad 30: Net-(D4-GK) -> Net-(U4-GPIO36)
- U4 pad 31: Net-(D5-RK) -> Net-(U4-GPIO38)
- U4 pad 32: Net-(D5-BK) -> Net-(U4-GPIO40)
Routing:
- net Net-(D3-BK): track 169.4 -> 11.3 mm, vias 5 -> 2
- net Net-(U4-GPIO34): track 0.00 -> 156.1 mm, vias 0 -> 3
- net Net-(J1-Pin_2): track 0.00 -> 125.2 mm, vias 0 -> 1
- net Net-(J1-Pin_1): track 0.00 -> 120.5 mm, vias 0 -> 1
- net Net-(D5-RK): track 53.6 -> 10.3 mm, vias 1 -> 0
- net Net-(U4-GPIO38): track 0.00 -> 41.7 mm, vias 0 -> 1
- net Net-(D3-RK): track 54.5 -> 17.1 mm, vias 3 -> 2
- net Net-(U4-GPIO21): track 0.00 -> 35.4 mm, vias 0 -> 1
- net Net-(D4-GK): track 46.8 -> 18.5 mm
- net Net-(U4-GPIO35): track 0.00 -> 26.5 mm, vias 0 -> 1
- net Net-(U4-GPIO36): track 0.00 -> 25.3 mm
- net Net-(D5-BK): track 63.5 -> 42.0 mm
- net Net-(U4-GPIO40): track 0.00 -> 19.9 mm
- net Net-(D5-GK): track 26.0 -> 8.10 mm, vias 1 -> 0
- net Net-(U4-GPIO39): track 0.00 -> 16.1 mm, vias 0 -> 1
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