File: Estacion/Estacion.kicad_sch (KiCad schematic)
At the start: 13 parts, among them SW1 SW_Push, U4 WeMos_S2_mini, U5 DHT22, U6 FN-M16P

Commit message: Emily me pega
Parts:
- D3, D4, D5: footprint LED_THT:LED_D5.0mm-4_RGB -> LED_THT:LED_D5.0mm-4_RGB_Wide_Pins
Changed lines of the file:
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@@
 			)
 		)
-		(property "Footprint" "LED_THT:LED_D5.0mm-4_RGB"
+		(property "Footprint" "LED_THT:LED_D5.0mm-4_RGB_Wide_Pins"
 			(at 73.66 72.39 0)
 			(hide yes)
@@
 			)
 		)
-		(property "Footprint" "LED_THT:LED_D5.0mm-4_RGB"
+		(property "Footprint" "LED_THT:LED_D5.0mm-4_RGB_Wide_Pins"
 			(at 73.66 113.03 0)
 			(hide yes)
@@
 			)
 		)
-		(property "Footprint" "LED_THT:LED_D5.0mm-4_RGB"
+		(property "Footprint" "LED_THT:LED_D5.0mm-4_RGB_Wide_Pins"
 			(at 73.66 91.44 0)
 			(hide yes)

Commit message: ?
Parts:
- removed LS2: Speaker, symbol Device:Speaker
- added J1: Conn_01x02_Pin, Connector_PinHeader_2.54mm:PinHeader_1x02_P2.54mm_Vertical, symbol Connector:Conn_01x02_Pin
- added R10, R4, R9: 220, Resistor_SMD:R_0805_2012Metric_Pad1.20x1.40mm_HandSolder, symbol Device:R
- added R11, R12, R5, R6, R7, R8: 150, Resistor_SMD:R_0805_2012Metric_Pad1.20x1.40mm_HandSolder, symbol Device:R
Connections:
- net at D3.1 (RK): now also R9.1; no longer U4.28 (GPIO21)
- net at D3.3 (BK): now also R7.1; no longer U4.29 (GPIO34)
- net at D3.4 (GK): now also R8.1; no longer U4.13 (GPIO33)
- net at U4.14 (GPIO35): now also R10.2; no longer D4.1 (RK)
- net at U4.15 (GPIO37): now also R11.1; no longer D4.3 (BK)
- net at U4.16 (GPIO39): now also R5.1; no longer D5.4 (GK)
- net at U4.30 (GPIO36): now also R12.1; no longer D4.4 (GK)
- net at U4.31 (GPIO38): now also R4.1; no longer D5.1 (RK)
- net at U4.32 (GPIO40): now also R6.1; no longer D5.3 (BK)
- net at U6.6 (SPK+): now also J1.1 (Pin_1)
- net at U6.8 (SPK-): now also J1.2 (Pin_2)
- new net: R8.2, U4.13 (GPIO33)
- new net: R9.2, U4.28 (GPIO21)
- new net: R7.2, U4.29 (GPIO34)
- new net: D5.1 (RK), R4.2
- new net: D5.3 (BK), R6.2
- new net: D5.4 (GK), R5.2
- new net: D4.1 (RK), R10.1
- new net: D4.3 (BK), R11.2
- new net: D4.4 (GK), R12.2
Other:
- moved on the sheet: D3, D5
